Commit message: Update robot description

File: src/hex_description/models/hex_model.xacro (robot description, xacro)
@@ -72,5 +72,5 @@
     </link>
     <joint name="tibia_joint_${side}${num}" type="revolute">
-        <origin xyz="0.08 0 0" rpy="0 0 0" />
+        <origin xyz="0.079 0 0" rpy="0 0 0" />
         <parent link="femur_${side}${num}" />
         <child link="tibia_${side}${num}" />
@@ -90,5 +90,5 @@
     </link>
     <joint name="tibia_foot_joint_${side}${num}" type="fixed">
-        <origin xyz="0.117 0 0" rpy="0 0 0" />
+        <origin xyz="0.129 0 0" rpy="0 0 0" />
         <parent link="tibia_${side}${num}" />
         <child link="tibia_foot_${side}${num}" />
